Commit message: created gazebo world and updted URDF

File: description/robot_core.xacro (robot description, xacro)
@@ -37,8 +37,11 @@
             </geometry>
         </collision>
-        <xacro:inertial_box mass="0.3" x="0.16" y="0.3" z="0.15">
+        <xacro:inertial_box mass="1.2" x="0.16" y="0.3" z="0.15">
         <origin xyz="0.08 0 0.03" rpy="0 0 0"/>
         </xacro:inertial_box>
     </link>
+<gazebo reference="chasis">
+    <material>Gazebo/White</material>
+</gazebo>
 <!--LEFT WHEEL LINK-->
 <joint name="left_wheel_joint" type="continuous"> <!-- continuous means it can rotate feeely unlike fixed link-->
@@ -51,5 +54,5 @@
     <visual>
         <geometry>
-            <cylinder radius="0.05" length="0.02" />
+            <cylinder radius="0.03" length="0.02" />
         </geometry>
         <material name="blue"/>
@@ -57,11 +60,14 @@
         <collision>
         <geometry>
-            <cylinder radius="0.05" length="0.02" />
+            <cylinder radius="0.03" length="0.02" />
         </geometry>
     </collision>
-    <xacro:inertial_cylinder mass="0.06" length="0.02" radius="0.05">
+    <xacro:inertial_cylinder mass="0.06" length="0.02" radius="0.03">
     <origin xyz ="0 0 0" rpy="0 0 0"/>
     </xacro:inertial_cylinder>
 </link>
+<gazebo reference="left_wheel">
+    <material>Gazebo/Blue</material>
+</gazebo>
 <!--RIGHT WHEEL LINK-->
 <joint name="right_wheel_joint" type="continuous"> <!-- continuous means it can rotate feeely unlike fixed link-->
@@ -74,5 +80,5 @@
     <visual>
         <geometry>
-            <cylinder radius="0.05" length="0.02" />
+            <cylinder radius="0.03" length="0.02" />
         </geometry>
         <material name="blue"/>
@@ -80,11 +86,14 @@
         <collision>
         <geometry>
-            <cylinder radius="0.05" length="0.02" />
+            <cylinder radius="0.03" length="0.02" />
         </geometry>
     </collision>
-        <xacro:inertial_cylinder mass="0.06" length="0.02" radius="0.05">
+        <xacro:inertial_cylinder mass="0.06" length="0.02" radius="0.03">
     <origin xyz ="0 0 0" rpy="0 0 0"/>
     </xacro:inertial_cylinder>
 </link>
+<gazebo reference="right_wheel">
+    <material>Gazebo/Blue</material>
+</gazebo>
 <!--CASTOR WHEEL LINK-->
 <joint name="castor_wheel_joint" type="fixed">
@@ -96,5 +105,5 @@
     <visual>
         <geometry>
-            <sphere radius="0.05"/>
+            <sphere radius="0.03"/>
         </geometry>
         <material name="black"/>
@@ -102,10 +111,15 @@
         <collision>
         <geometry>
-            <sphere radius="0.05"/>
+            <sphere radius="0.03"/>
         </geometry>
     </collision>
-    <xacro:inertial_sphere mass="0.01" radius="0.05">
+    <xacro:inertial_sphere mass="0.1" radius="0.03">
     <origin xyz ="0 0 0" rpy="0 0 0"/>
     </xacro:inertial_sphere>
 </link>
+<gazebo reference="castor_wheel">
+    <material>Gazebo/Black</material>
+    <mu1 value="0.001"/>
+    <mu2 value="0.001"/>
+</gazebo>
 </robot>
