Commit message: added tracker ball model in gazebo world

File: description/robot.urdf.xacro (robot description, xacro)
@@ -3,3 +3,4 @@
    <xacro:include filename="robot_core.xacro" />
    <xacro:include filename="gazebo_control.xacro"/>
+   <xacro:include filename="camera.xacro"/>
 </robot>

File: description/robot_core.xacro (robot description, xacro)
@@ -48,5 +48,5 @@
     <parent link="base_link"/>
     <child  link="left_wheel"/>
-    <origin xyz="-0.03 0.09 0" rpy="-${pi/2} 0 0"/>
+    <origin xyz="-0.045 0.09 0" rpy="-${pi/2} 0 0"/>
     <axis xyz="0 0 1"/>
 </joint>
@@ -74,5 +74,5 @@
     <parent link="base_link"/>
     <child  link="right_wheel"/>
-    <origin xyz="-0.03 -0.09 0" rpy="${pi/2} 0 0"/>
+    <origin xyz="-0.045 -0.09 0" rpy="${pi/2} 0 0"/>
     <axis xyz="0 0 -1"/>
 </joint>
@@ -114,5 +114,5 @@
         </geometry>
     </collision>
-    <xacro:inertial_sphere mass="0.1" radius="0.03">
+    <xacro:inertial_sphere mass="0.08" radius="0.03">
     <origin xyz ="0 0 0" rpy="0 0 0"/>
     </xacro:inertial_sphere>
@@ -120,6 +120,6 @@
 <gazebo reference="castor_wheel">
     <material>Gazebo/Black</material>
-    <mu1 value="0.001"/>
-    <mu2 value="0.001"/>
-</gazebo>
+    <mu1 value="0.0015"/>
+    <mu2 value="0.0015"/>
+    </gazebo>
 </robot>
